Commit message: Prawie działąjące move goal

File: cyber_is_description/urdf/cyber_is.xacro (robot description, xacro)
@@ -274,5 +274,5 @@
     <!-- Umieszczenie skanera na środku ramy (x=0,y=0) i na wysokości scan_height nad podłożem.
          Base_link jest track_center_height nad podłożem, więc offset względem base_link to (scan_height - track_center_height). -->
-    <origin xyz="0 0 ${scan_height - chassis_top_height}" rpy="0 0 0"/>
+    <origin xyz="0 0 ${scan_height - chassis_top_height}" rpy="0 0 3.14159"/>
     <parent link="base_link"/>
     <child link="base_scan"/>

Commit message: add supervisor.py

File: cyber_is_description/urdf/cyber_is.xacro (robot description, xacro)
@@ -274,5 +274,5 @@
     <!-- Umieszczenie skanera na środku ramy (x=0,y=0) i na wysokości scan_height nad podłożem.
          Base_link jest track_center_height nad podłożem, więc offset względem base_link to (scan_height - track_center_height). -->
-    <origin xyz="0 0 ${scan_height - chassis_top_height}" rpy="0 0 3.14159"/>
+    <origin xyz="0 0 ${scan_height - chassis_top_height}" rpy="0 0 0"/>
     <parent link="base_link"/>
     <child link="base_scan"/>

Commit message: add supervisor.py

File: cyber_is_description/urdf/cyber_is.xacro (robot description, xacro)
@@ -181,5 +181,5 @@
     <visual>
       <!-- Cylinder pionowy reprezentujący skaner -->
-      <origin xyz="0 0 0" rpy="0 0 0"/>
+      <origin xyz="0 0 0" rpy="0 0 3.14159"/>
       <geometry>
         <cylinder radius="0.03" length="0.025"/>

Commit message: add supervisor.py

File: cyber_is_description/urdf/cyber_is.xacro (robot description, xacro)
@@ -214,5 +214,5 @@
   <joint name="base_link_joint" type="fixed">
     <!-- base_link znajduje się track_center_height nad base_footprint (z = 0.03 m) -->
-    <origin xyz="0 0 ${chassis_top_height}" rpy="0 0 0"/>
+    <origin xyz="0 0 ${chassis_top_height}" rpy="0 0 3.14159"/>
     <parent link="base_footprint"/>
     <child link="base_link"/>

Commit message: upgrade navigation

File: cyber_is_description/urdf/cyber_is.xacro (robot description, xacro)
@@ -274,5 +274,5 @@
     <!-- Umieszczenie skanera na środku ramy (x=0,y=0) i na wysokości scan_height nad podłożem.
          Base_link jest track_center_height nad podłożem, więc offset względem base_link to (scan_height - track_center_height). -->
-    <origin xyz="0 0 ${scan_height - chassis_top_height}" rpy="0 0 3.14159"/>
+    <origin xyz="0.02 0 ${scan_height - chassis_top_height}" rpy="0 0 3.14159"/>
     <parent link="base_link"/>
     <child link="base_scan"/>

Commit message: fix

File: cyber_is_description/urdf/cyber_is.xacro (robot description, xacro)
@@ -219,6 +219,6 @@
   </joint>
   <!-- Połączenia (joints) między linkami -->
-  <!-- Stałe połączenie base_link (na ziemi) z imu (ramą) -->
-  <joint name="imu_joint" type="continuous">
+  <!-- Stałe połączenie base_link z imu (ramą) -->
+  <joint name="imu_joint" type="fixed">
     <!-- Pozycja: z przodu (x = +half długości), na lewo (y = +half rozstawu), na wysokości osi (z = track_center_height) -->
     <origin xyz="0 0 0" rpy="0 0 0"/>
@@ -227,7 +227,6 @@
     <!-- Oś obrotu: pozioma, w poprzek pojazdu (oś Y układu bazowego) -->
   </joint>
-  <!-- Połączenia (joints) między linkami -->
-  <!-- Stałe połączenie base_link (na ziemi) z imu (ramą) -->
-  <joint name="line_detector_joint" type="continuous">
+  <!-- Połączenie stałe base_link z line_detector -->
+  <joint name="line_detector_joint" type="fixed">
     <!-- Pozycja: z przodu (x = +half długości), na lewo (y = +half rozstawu), na wysokości osi (z = track_center_height) -->
     <origin xyz="${frame_length/2 +0.005} 0 -${chassis_height}" rpy="0 0 0"/>
